Commit message: change urdf with real mesh file

File: description/robot_core.xacro (robot description, xacro)
@@ -2,4 +2,5 @@
 <robot xmlns:xacro="http://www.ros.org/wiki/xacro" >
     <xacro:include filename="inertial_macros.xacro"/>
+   <xacro:property name="scale_ratio" value="0.0015" />
     <material name="white">
         <color rgba="1 1 1 1" />
@@ -25,14 +26,14 @@
     <link name="chassis">
         <visual>
-            <origin xyz="0.15 0 0.05"/>
+            <origin xyz="0 0.15 0" rpy="1.57 0 0"/>
             <geometry>
-                <box size="0.3 0.2 0.10"/>
+                <mesh scale="${scale_ratio} ${scale_ratio} ${scale_ratio}" filename="file:///home/samet/Desktop/develop/education_robot_ws/src/education_robot/description/meshes/body.stl" />
             </geometry>
             <material name="white"/>
         </visual>
         <collision>
-            <origin xyz="0.15 0 0.075"/>
+            <origin xyz="0.25 0 0.075"/>
             <geometry>
-                <box size="0.3 0.3 0.15"/>
+                <box size="0.5 0.3 0.15"/>
             </geometry>
         </collision>
@@ -45,5 +46,5 @@
         <parent link="base_link"/>
         <child link="left_wheel"/>
-        <origin xyz="0.05 0.14 0" rpy="-${pi/2} 0 0" />
+        <origin xyz="0.145 0.14 0.04" rpy="-${pi/2} 0 0" />
         <axis xyz="0 0 1"/>
     </joint>
@@ -51,7 +52,8 @@
         <visual>
             <geometry>
-                <cylinder radius="0.04" length="0.04"/>
+                <mesh scale="${scale_ratio} ${scale_ratio} ${scale_ratio}" filename="file:///home/samet/Desktop/develop/education_robot_ws/src/education_robot/description/meshes/wheel.stl" />
             </geometry>
             <material name="blue"/>
+            <origin xyz="-0.049 -0.049 0" rpy="0 ${pi/2} 0" />
         </visual>
         <collision>
@@ -68,5 +70,5 @@
         <parent link="base_link"/>
         <child link="right_wheel"/>
-        <origin xyz="0.05 -0.14 0" rpy="${pi/2} 0 0" />
+        <origin xyz="0.145 -0.14 0.04" rpy="-${pi/2} 0 0" />
         <axis xyz="0 0 -1"/>
     </joint>
@@ -74,6 +76,7 @@
         <visual>
             <geometry>
-                <cylinder radius="0.04" length="0.04"/>
+                <mesh scale="${scale_ratio} ${scale_ratio} ${scale_ratio}" filename="file:///home/samet/Desktop/develop/education_robot_ws/src/education_robot/description/meshes/wheel.stl" />
             </geometry>
+            <origin xyz="-0.049 -0.049 0" rpy="0 ${pi/2} 0" />
             <material name="blue"/>
         </visual>
@@ -87,6 +90,29 @@
         </xacro:inertial_cylinder>
     </link>
+    <joint name="lidar_joint" type="fixed">
+        <parent link="chassis"/>
+        <child link="lidar_link"/>
+        <origin xyz="0.4 0 0.2"/>
+    </joint>
+    <link name="lidar_link">
+        <visual>
+            <origin xyz="-0.05 0.03 -0.02" rpy="1.57 0 0"/>
+            <geometry>
+                <mesh scale="${scale_ratio} ${scale_ratio} ${scale_ratio}" filename="file:///home/samet/Desktop/develop/education_robot_ws/src/education_robot/description/meshes/lidar.stl" />
+            </geometry>
+            <material name="orange"/>
+        </visual>
+        <collision>
+            <origin xyz="0 0 0"/>
+            <geometry>
+                <box size="0.05 0.05 0.05"/>
+            </geometry>
+        </collision>
+        <xacro:inertial_box mass="0.1" x="0.05" y="0.05" z="0.05">
+            <origin xyz="0.15 0 0.075" rpy="0 0 0"/>
+        </xacro:inertial_box>
+    </link>
     <!-- CASTER WHEEL LINK -->
-    <joint name="caster_wheel_joint" type="fixed">
+  <!--  <joint name="caster_wheel_joint" type="fixed">
         <parent link="chassis"/>
         <child link="caster_wheel"/>
@@ -130,3 +156,4 @@
         </xacro:inertial_sphere>
     </link>
+    -->
 </robot>
