Commit message: add gazebo control

File: description/robot.urdf.xacro (robot description, xacro)
@@ -3,3 +3,4 @@
     <!-- Example link -->
     <xacro:include filename="robot_core.xacro"/>
+    <xacro:include filename="gazebo_control.xacro"/>
 </robot>

File: description/robot_core.xacro (robot description, xacro)
@@ -42,4 +42,7 @@
         </xacro:inertial_box>
     </link>
+    <gazebo reference="chassis">
+    <material>Gazebo/Gray</material>
+    </gazebo>
     <!-- LEFT WHEEL LINK -->
     <joint name="left_wheel_joint" type="continuous">
@@ -66,4 +69,7 @@
         </xacro:inertial_cylinder>
     </link>
+    <gazebo reference="left_wheel">
+    <material>Gazebo/Black</material>
+    </gazebo>
     <!-- RIGHT WHEEL LINK -->
     <joint name="right_wheel_joint" type="continuous">
@@ -71,5 +77,5 @@
         <child link="right_wheel"/>
         <origin xyz="0.145 -0.14 0.04" rpy="-${pi/2} 0 0" />
-        <axis xyz="0 0 -1"/>
+        <axis xyz="0 0 1"/>
     </joint>
     <link name="right_wheel">
@@ -90,4 +96,7 @@
         </xacro:inertial_cylinder>
     </link>
+    <gazebo reference="right_wheel">
+    <material>Gazebo/Black</material>
+    </gazebo>
     <joint name="lidar_joint" type="fixed">
         <parent link="chassis"/>
@@ -113,4 +122,7 @@
         </xacro:inertial_box>
     </link>
+    <gazebo reference="lidar_link">
+    <material>Gazebo/Black</material>
+    </gazebo>
     <!-- CASTER WHEEL LINK -->
   <!--  <joint name="caster_wheel_joint" type="fixed">
